File: MultiROM.kicad_pcb (KiCad board)
At the start: 2 copper layers, 85.1 x 62.9 mm, 7 parts, among them J1 Conn_02x22_Row_Letter_First, SW1 SW_DIP_x04, U1 SST39SF010, U2 GAL16V8

Commit message: PCB revisions post proto#1
Parts:
- C1: moved to B.Cu
- U1: footprint Package_DIP:DIP-32_W15.24mm_Socket -> Package_DIP:DIP-32_W15.24mm
- turned C1 to 180 degrees
Connections:
- RN1 pad 3: /~{Hi_A16} -> /~{Lo_A15}
- RN1 pad 4: /~{Hi_A15} -> /~{Lo_A16}
- RN1 pad 5: /~{Lo_A16} -> /~{Hi_A15}
- RN1 pad 6: /~{Lo_A15} -> /~{Hi_A16}
- SW1 pad 1: /~{Hi_A16} -> /~{Lo_A15}
- SW1 pad 2: /~{Hi_A15} -> /~{Lo_A16}
- SW1 pad 3: /~{Lo_A16} -> /~{Hi_A15}
- SW1 pad 4: /~{Lo_A15} -> /~{Hi_A16}
- U2 pad 6: /~{Lo_A15} -> /~{Hi_A16}
- U2 pad 7: /~{Lo_A16} -> /~{Hi_A15}
- U2 pad 8: /~{Hi_A15} -> /~{Lo_A16}
- U2 pad 9: /~{Hi_A16} -> /~{Lo_A15}
Routing:
- net /~{Hi_A16}: track 26.1 -> 36.0 mm
- net /~{Lo_A15}: track 36.0 -> 26.1 mm
- net /D3: track 48.8 -> 54.6 mm
- net /~{Lo_A16}: track 32.4 -> 28.8 mm
- net /~{Hi_A15}: track 28.8 -> 32.4 mm
Other:
- outline, holes or cut-outs redrawn
- board text added: "128K flash ROM catridge for BBC Master and Acorn Electron"
- board text added: "MultiROM"
- board text added: "github.com/rhalkyard/bbc-multirom Issue 1"
- board text removed: "A1"
- board text removed: "A22"
- board text removed: "B1"
- board text removed: "B22"
- board text removed: "JLCJLCJLCJLC"
