File: MultiROM.kicad_sch (KiCad schematic)
At the start: 7 parts, among them J1 Conn_02x22_Row_Letter_First, SW1 SW_DIP_x04, U1 SST39SF010, U2 GAL16V8

Commit message: PCB revisions post proto#1
Parts:
- U1: footprint Package_DIP:DIP-32_W15.24mm_Socket -> Package_DIP:DIP-32_W15.24mm
Connections:
- net ~{Hi_A15}: now also RN1.5 (R4), SW1.3, U2.7 (I7); no longer RN1.4 (R3), SW1.2, U2.8 (I8)
- net ~{Hi_A16}: now also RN1.6 (R5), SW1.4, U2.6 (I6); no longer RN1.3 (R2), SW1.1, U2.9 (I9)
- net ~{Lo_A15}: now also RN1.3 (R2), SW1.1, U2.9 (I9); no longer RN1.6 (R5), SW1.4, U2.6 (I6)
- net ~{Lo_A16}: now also RN1.4 (R3), SW1.2, U2.8 (I8); no longer RN1.5 (R4), SW1.3, U2.7 (I7)
Changed lines of the file:
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@@
     (effects (font (size 1.27 1.27)) (justify right bottom))
   )
-  (label "~{Hi_A15}" (at 151.13 121.92 0) (fields_autoplaced)
+  (label "~{Hi_A15}" (at 151.13 119.38 0) (fields_autoplaced)
     (effects (font (size 1.27 1.27)) (justify left bottom))
   )
@@
     (effects (font (size 1.27 1.27)) (justify right bottom))
   )
-  (label "~{Lo_A15}" (at 151.13 116.84 0) (fields_autoplaced)
+  (label "~{Lo_A15}" (at 151.13 124.46 0) (fields_autoplaced)
     (effects (font (size 1.27 1.27)) (justify left bottom))
   )
@@
     (effects (font (size 1.27 1.27)) (justify right bottom))
   )
-  (label "~{Hi_A16}" (at 151.13 124.46 0) (fields_autoplaced)
+  (label "~{Hi_A16}" (at 151.13 116.84 0) (fields_autoplaced)
     (effects (font (size 1.27 1.27)) (justify left bottom))
   )
@@
     (effects (font (size 1.27 1.27)) (justify right bottom))
   )
-  (label "~{Lo_A16}" (at 151.13 119.38 0) (fields_autoplaced)
+  (label "~{Lo_A16}" (at 151.13 121.92 0) (fields_autoplaced)
     (effects (font (size 1.27 1.27)) (justify left bottom))
   )
@@
       (effects (font (size 1.27 1.27)))
     )
-    (property "Footprint" "Package_DIP:DIP-32_W15.24mm_Socket" (at 44.45 109.22 0)
-      (effects (font (size 1.27 1.27)) hide)
-    )
+    (property "Footprint" "Package_DIP:DIP-32_W15.24mm" (at 44.45 109.22 0)
+      (effects (font (size 1.27 1.27)) hide)
+    )
