File: pcb/MultiROM.kicad_sch (KiCad schematic)
At the start: 7 parts, among them J1 Conn_02x22_Row_Letter_First, SW1 SW_DIP_x04, U1 SST39SF010, U2 GAL16V8

Commit message: PCB+netlist tidyup
Connections:
- net ~{Hi_A15}: now also RN1.6 (R5), SW1.4, U2.6 (I6); no longer RN1.5 (R4), SW1.3, U2.7 (I7)
- net ~{Hi_A16}: now also RN1.5 (R4), SW1.3, U2.7 (I7); no longer RN1.6 (R5), SW1.4, U2.6 (I6)
- net ~{Lo_A15}: now also RN1.4 (R3), SW1.2, U2.8 (I8); no longer RN1.3 (R2), SW1.1, U2.9 (I9)
- net ~{Lo_A16}: now also RN1.3 (R2), SW1.1, U2.9 (I9); no longer RN1.4 (R3), SW1.2, U2.8 (I8)
- net CS_R~{W} renamed R~{W}_{E}_CS_{M}
- net M_R~{W} renamed R~{W}_{M}
Other:
- moved on the sheet: C1, C2, J1, RN1, SW1, U1, U2

Commit message: Rename cartridge footprint+library to avoid spaces
Parts:
- J1: footprint BBC Master Cartridge:BBC Master Cartridge -> BBC Master / Acorn Electron Cartridge:bbc-master-acorn-electron-cartridge
Changed lines of the file:
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@@
       (effects (font (size 1.27 1.27)))
     )
-    (property "Footprint" "BBC Master Cartridge:BBC Master Cartridge" (at 31.75 45.085 0)
+    (property "Footprint" "BBC Master / Acorn Electron Cartridge:bbc-master-acorn-electron-cartridge" (at 31.75 45.085 0)
       (effects (font (size 1.27 1.27)) hide)
     )
