File: pcb/MultiROM.kicad_pcb (KiCad board)
At the start: 2 copper layers, 85.1 x 62.9 mm, 7 parts, among them J1 Conn_02x22_Row_Letter_First, SW1 SW_DIP_x04, U1 SST39SF010, U2 GAL16V8

Commit message: Issue 1
Other:
- board text added: "github.com/rhalkyard/bbc-multirom Issue 1"
- board text removed: "github.com/rhalkyard/bbc-multirom"
Changed lines of the file:
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@@
     (effects (font (size 1 1) (thickness 0.15)))
   )
-  (gr_text "github.com/rhalkyard/bbc-multirom\n" (at 36.195 57.785 90) (layer "F.SilkS")
+  (gr_text "github.com/rhalkyard/bbc-multirom\nIssue 1" (at 36.195 57.785 90) (layer "F.SilkS")
     (effects (font (size 1 1) (thickness 0.125)) (justify left top))
   )
